Commit message: model changes, still no textures on mesh

File: sdpp_human_description/urdf/person.urdf (robot description, URDF)
Before this commit: robot person, 2 links, 1 joints
Links:
- link base_link: geometry collision box size=.5 .5 .2; visual mesh filename=package://sdpp_human_description/meshes/standing.dae
