Commit message: cleanup commit

File: sdpp_human_description/urdf/diff_human.urdf.xacro (robot description, xacro)
@@ -135,5 +135,5 @@
     <parent link="base_link"/>
     <child link="base_scan"/>
-    <origin xyz="-0.064 0 1.0" rpy="0 0 0"/>
+    <origin xyz="-0.064 0 0.5" rpy="0 0 0"/>
   </joint>
   <link name="base_scan">
